File: car_amp_analog_mono/car_amp_analog_mono.sch (KiCad schematic (older format))
At the start: 20 parts, among them U1 L7805, U2 NE5532

Commit message: Add Audio Input Buffer
Parts:
- added C?: 4.7u, symbol Device:C
- added C?: 1n, symbol Device:C
- added C?: 100n, symbol Device:C
- added FB?: 600 @ 600 MHz, symbol Device:Ferrite_Bead_Small
- added R? (x2): 10R, symbol Device:R
- added R? (x2): 22K, symbol Device:R
- added R?: 100R, symbol Device:R
- added U4: NE5532, symbol Amplifier_Operational:NE5532
- gave numbers to parts that had none: 1
Connections:
- net labels added: AUDIO_IN, INP_BUF_OUT
- wire segments 74 -> 115
Other:
- note added: "Audio Input Buffer"
- moved on the sheet: C1, C2, C3, C4, C?, Q?, R1, R?, U1, U2B, U2C

Commit message: Add Volume Control
Parts:
- removed U?: ATmega328P-PU, Package_DIP:DIP-28_W7.62mm, symbol MCU_Microchip_ATmega:ATmega328P-PU
- added C?: 220u, symbol Device:CP
- added C?: C, symbol Device:C
- added C? (x3): 100p, symbol Device:C
- added R? (x2): 10, symbol Device:R
- added R?: 47k, symbol Device:R
- added R? (x4): 1K, symbol Device:R
- added R? (x3): 5K6, symbol Device:R
- added R?: R, symbol Device:R
- added R?: 1k, symbol Device:R
- added U? (x4): NE5532, symbol Amplifier_Operational:NE5532
- added U?: MCP41010, symbol Potentiometer_Digital:MCP41010
- R1: value 12K -> 12k
- R?: value 3.3K -> 3k3
- R?: value 1.1K -> 1k1
- R? (x4): value 10R -> 10
- R? (x2): value 2.2K -> 2k2
- R? (x2): value 22K -> 22k
- R?: value 100R -> 100
Connections:
- net labels added: VAS_OUT
- wire segments 115 -> 187
Other:
- note added: "Volume Control"

Commit message: Add Pre-Driver
Parts:
- added C?: 10u, symbol Device:C
- added C?: 100n, symbol Device:C
- added R? (x2): 10, symbol Device:R
- added R?: 22k, symbol Device:R
- added U? (x3): NE5532, symbol Amplifier_Operational:NE5532
- C?: value C -> 10u
- R?: value R -> 3k3
- gave numbers to parts that had none: 2
- renumbered U4 to U3, U3 to U?
Connections:
- net labels added: PRE_DRIVE_OUT, VOL_CTR_OUT
- net labels removed: VAS_OUT
- wire segments 187 -> 220
Other:
- note added: "Pre-Driver"
- moved on the sheet: C?, R?, U4A, U5A, U5B

Commit message: Add Power Amp (with library)
Parts:
- added C?: 2200u, symbol Device:CP
- added C? (x3): 100n, symbol Device:C
- added C?: 1000u, symbol Device:CP
- added C?: 47u, symbol Device:CP
- added C?: 10u, symbol Device:CP
- added R?: 10, symbol Device:R
- added R? (x2): 10k, symbol Device:R
- added R? (x4): 1, symbol Device:R
- added U? (x6): NE5532, symbol Amplifier_Operational:NE5532
- added U?: TDA7377A, footprints:Multiwatt-15, symbol car_amp:TDA7377A
Connections:
- net labels added: DRIVER_OUT, HP_OUT, ST-BY
- wire segments 220 -> 311
Other:
- note added: "Drivers"
- note added: "Output Protection and Filtering"
- note added: "Power Amp"
